File: battery_load_tester_v1.0/battery_load_tester.kicad_pcb (KiCad board)
At the start: 2 copper layers, 69.1 x 53.8 mm, 6 parts, among them J1 Screw Terminal (Arduino Power), J2 Screw Terminal (Test Battery), J3 MicroSD Reader

Commit message: v1 updated and printed
Parts:
- moved R1 5.08 mm to (161.8, 82.0)
- moved C1 2.72 mm to (117.1, 78.2), turned to 180 degrees
Routing:
- net Earth: track 0.00 -> 11.7 mm
- net Net-(A1-Pad9): track 39.4 -> 34.3 mm
- net +3V3: track 66.1 -> 67.2 mm
Other:
- board text added: "Battery Load Tester (v1.0)"
- board text removed: "Battery Tester v1.0"
